Commit message: Modifying needed files and adding new VR testing script

File: iGibson/needed_files/nico_upper_head_rh6d_dual.urdf (robot description, URDF)
Before this commit: robot nico_upper_rh6d, 21 links, 20 joints
Links:
- added link littlefingel, mass 0.000009; collision mesh filename=mesh/finger.stl; visual mesh filename=mesh/finger.obj
- added link littlefinger, mass 0.000009; collision mesh filename=mesh/finger.stl; visual mesh filename=mesh/finger.obj
- added link middlefingel, mass 0.000009; collision mesh filename=mesh/finger.stl; visual mesh filename=mesh/finger.obj
- added link middlefinger, mass 0.000009; collision mesh filename=mesh/finger.stl; visual mesh filename=mesh/finger.obj
- link endeffector: mass None -> 0.000009
Joints:
- added joint litlefingel_rjoint: type revolute, parent left_palm, child littlefingel, origin xyz=0.00 0.02 -0.06 rpy=0 0 0, axis 0 1 0, limit lower=0 upper=2.57 effort=30 velocity=1
- added joint litlefinger_rjoint: type revolute, parent right_palm, child littlefinger, origin xyz=0.00 0.02 -0.06 rpy=0 0 0, axis 0 1 0, limit lower=-2.57 upper=0 effort=30 velocity=1
- added joint middlefingel_rjoint: type revolute, parent left_palm, child middlefingel, origin xyz=0 0 -0.06 rpy=0 0 0, axis 0 1 0, limit lower=0 upper=2.57 effort=30 velocity=1
- added joint middlefinger_rjoint: type revolute, parent right_palm, child middlefinger, origin xyz=0 0 -0.06 rpy=0 0 0, axis 0 1 0, limit lower=-2.57 upper=0 effort=30 velocity=1

Commit message: Right hand grabbing

File: iGibson/needed_files/nico_upper_head_rh6d_dual.urdf (robot description, URDF)
Before this commit: robot nico_upper_rh6d, 25 links, 24 joints
Joints:
- removed joint litlefingel_rjoint
- removed joint litlefinger_rjoint
- added joint littlefingel_rjoint: type revolute, parent left_palm, child littlefingel, origin xyz=0.00 0.02 -0.06 rpy=0 0 0, axis 0 1 0, limit lower=0 upper=2.57 effort=30 velocity=1
- added joint littlefinger_rjoint: type revolute, parent right_palm, child littlefinger, origin xyz=0.00 0.02 -0.06 rpy=0 0 0, axis 0 1 0, limit lower=-2.57 upper=0 effort=30 velocity=1

Commit message: WIP

File: iGibson/needed_files/nico_upper_head_rh6d_dual.urdf (robot description, URDF)
Before this commit: robot nico_upper_rh6d, 25 links, 24 joints
Links:
- link endeffectol: mass None -> 0.000009
